File: Kicad Files/left.kicad_sch (KiCad schematic)
At the start: 51 parts, among them J1 PJ-320A-DoubleSide, SW22 PCM12SMTR, U2 Universal_Pro_Micro

Commit message: Xiao Controller
Parts:
- removed J1: PJ-320A-DoubleSide, Keebio-Parts:TRRS-PJ-320A, symbol ClaudeSym:PJ-320A
- removed RSW1: SW_PUSH, ClaudeFoot:ResetSW_1side, symbol kbd:SW_PUSH
- removed U2: Universal_Pro_Micro, ClaudeFoot:Universal_Pro_Micro_Footprint, symbol ClaudeSym:Universal_Pro_Micro_Footprint
- added J2: BATl, Connector_JST:JST_GH_SM02B-GHS-TB_1x02-1MP_P1.25mm_Horizontal, symbol Connector_Generic:Conn_01x02
- added U3: Seeed Studio XIAO nRF52840, Kicad Files:XIAO-nRF52840-Sense-14P-2.54-21X17.8MM_custom, symbol Xiao:Seeed Studio XIAO nRF52840
- BT1, BT2, BT3, BT4: footprint ClaudeFoot:Breakaway_Tabs -> kbd:Breakaway_Tabs
- SW? (x20): footprint ClaudeFoot:SW_MXchoc_HS_1u -> kbd:keyswitch_choc12_hotswap_1u
- SW?: footprint ClaudeFoot:SW_MXchoc_HS_1u -> kbd:keyswitch_choc12_hotswap_1.5u
Connections:
- net B- renamed -BATTl
- net -BATTl: now also J2.2 (Pin_2)
- net GND renamed GNDl
- net GNDl: now also U3.13 (GND), U3.21 (BAT-)
- net MOSI renamed SDAl
- net SDAl: now also U3.5 (P0.04_A4_D4_SDA)
- net SCK renamed SCLl
- net SCLl: now also U3.6 (P0.05_A5_D5_SCL)
- net VCC renamed VCCl
- net VCCl: now also U3.12 (3V3)
- net col0 renamed col0l
- net col0l: now also U3.20 (P0.10_NFC2)
- net col1 renamed col1l
- net col1l: now also U3.11 (P1.15_D10_MOSI)
- net col2 renamed col2l
- net col2l: now also U3.10 (P1.14_D9_MISO)
- net col3 renamed col3l
- net col3l: now also U3.9 (P1.13_D8_SCK)
- net col4 renamed col4l
- net col4l: now also U3.8 (P1.12_D7_RX)
- net col5 renamed col5l
- net col5l: now also U3.7 (P1.11_D6_TX)
- net cs renamed csl
- net csl: now also U3.19 (P0.09_NFC1)
- net row0 renamed row0l
- net row0l: now also U3.1 (P0.02_A0_D0)
- net row1 renamed row1l
- net row1l: now also U3.2 (P0.03_A1_D1)
- net row2 renamed row2l
- net row2l: now also U3.3 (P0.28_A2_D2)
- net row3 renamed row3l
- net row3l: now also U3.4 (P0.29_A3_D3)
- new net +BATTl: J2.1 (Pin_1), U3.22 (BAT+)
- no-connect marks 6 -> 5
Other:
- moved on the sheet: SW22
