File: Kicad Files/right.kicad_sch (KiCad schematic)
At the start: 51 parts, among them J2 PJ-320A-DoubleSide, SW44 PCM12SMTR, U1 Universal_Pro_Micro

Commit message: Xiao Controller
Parts:
- removed J2: PJ-320A-DoubleSide, Keebio-Parts:TRRS-PJ-320A, symbol ClaudeSym:PJ-320A
- removed RSW2: SW_PUSH, ClaudeFoot:ResetSW_1side, symbol kbd:SW_PUSH
- removed U1: Universal_Pro_Micro, ClaudeFoot:Universal_Pro_Micro_Footprint, symbol ClaudeSym:Universal_Pro_Micro_Footprint
- added J1: BATr, Connector_JST:JST_GH_SM02B-GHS-TB_1x02-1MP_P1.25mm_Horizontal, symbol Connector_Generic:Conn_01x02
- added U2: Seeed Studio XIAO nRF52840, Kicad Files:XIAO-nRF52840-Sense-14P-2.54-21X17.8MM_custom, symbol Xiao:Seeed Studio XIAO nRF52840
- rBT1, rBT2, rBT3, rBT4: footprint ClaudeFoot:Breakaway_Tabs -> kbd:Breakaway_Tabs
- rSW? (x18): footprint ClaudeFoot:SW_MXchoc_HS_1u -> kbd:keyswitch_choc12_hotswap_1u
- rSW? (x2): footprint ClaudeFoot:SW_MXchoc_HS_1u -> Kicad Files:keyswitch_choc12_hotswap_1u
- rSW?: footprint ClaudeFoot:SW_MXchoc_HS_1u -> kbd:keyswitch_choc12_hotswap_1.5u
Connections:
- net GNDr: now also U2.13 (GND), U2.21 (BAT-)
- net VCCr: now also U2.12 (3V3)
- net col0r: now also U2.20 (P0.10_NFC2)
- net col1r: now also U2.11 (P1.15_D10_MOSI)
- net col2r: now also U2.10 (P1.14_D9_MISO)
- net col3r: now also U2.9 (P1.13_D8_SCK)
- net col4r: now also U2.8 (P1.12_D7_RX)
- net col5r: now also U2.7 (P1.11_D6_TX)
- net csr: now also U2.19 (P0.09_NFC1)
- net row0r: now also U2.1 (P0.02_A0_D0)
- net row1r: now also U2.2 (P0.03_A1_D1)
- net row2r: now also U2.3 (P0.28_A2_D2)
- net row3r: now also U2.4 (P0.29_A3_D3)
- net -BATTr: now reaches SW44.3
- net -BATTr: now also J1.2 (Pin_2)
- net B-r: no longer names the net of SW44.1
- net MOSIr renamed SDAr
- net SDAr: now also U2.5 (P0.04_A4_D4_SDA)
- net SCKr renamed SCLr
- net SCLr: now also U2.6 (P0.05_A5_D5_SCL)
- new net +BATTr: J1.1 (Pin_1), U2.22 (BAT+)
